Commit message: add special connection to urdfs

File: franka_description/robots/panda_arm.urdf.xacro (robot description, xacro)
@@ -6,9 +6,45 @@
   <xacro:arg name="use_fake_hardware" default="false"/>
   <xacro:arg name="fake_sensor_commands" default="false"/>
+  <xacro:arg name="special_connection" default=""/> <!-- Connection between the arm and the end-effector -->
+  <xacro:property name="special_connection" value="$(arg special_connection)"/>
   <xacro:include filename="$(find franka_description)/robots/panda_arm.xacro"/>
   <xacro:panda_arm arm_id="$(arg arm_id)" safety_distance="0.03"/>
+  <xacro:if value="${special_connection == ''}">
+    <xacro:property name="ee_xyz" value="0 0 0"/>
+    <xacro:property name="ee_rpy" value="0 0 ${-pi/4}"/>
+    <xacro:property name="ee_connected_to" value="$(arg arm_id)_link8"/>
+  </xacro:if>
+  <xacro:unless value="${special_connection == ''}">
+    <link name="${special_connection}">
+      <xacro:if value="${special_connection == 'robotiq_ft_sensor'}">
+        <visual>
+          <geometry>
+            <mesh filename="package://franka_description/meshes/accessories/robotiq_ft_300.stl" />
+          </geometry>
+          <material name="black">
+            <color rgba="0.1 0.1 0.1 1"/>
+          </material>
+        </visual>
+        <collision>
+          <geometry>
+            <mesh filename="package://franka_description/meshes/accessories/robotiq_ft_300.stl" />
+          </geometry>
+        </collision>
+      </xacro:if>
+    </link>
+    <joint name="${special_connection}_joint" type="fixed">
+      <parent link="$(arg arm_id)_link8"/>
+      <child link="${special_connection}"/>
+      <xacro:if value="${special_connection == 'robotiq_ft_sensor'}">
+        <origin xyz="0 0 0.0375" rpy="0 0 ${pi/2}"/>
+      </xacro:if>
+    </joint>
+    <xacro:property name="ee_xyz" value="0 0 0.002"/>
+    <xacro:property name="ee_rpy" value="0 0 ${(5/4)*pi}"/>
+    <xacro:property name="ee_connected_to" value="${special_connection}"/>
+  </xacro:unless>
   <xacro:if value="$(arg hand)">
     <xacro:include filename="$(find franka_description)/robots/hand.xacro"/>
-    <xacro:hand ns="$(arg arm_id)" rpy="0 0 ${-pi/4}" connected_to="$(arg arm_id)_link8" safety_distance="0.03"/>
+    <xacro:hand ns="$(arg arm_id)" xyz="${ee_xyz}" rpy="${ee_rpy}" connected_to="${ee_connected_to}" safety_distance="0.03"/>
   </xacro:if>
   <xacro:include filename="$(find franka_description)/robots/panda_arm.ros2_control.xacro"/>

File: franka_moveit_config/srdf/panda_arm.srdf.xacro (robot description, xacro)
@@ -3,12 +3,13 @@
   <xacro:arg name="arm_id" default="panda"/> <!-- Name of this panda -->
   <xacro:arg name="hand" default="true"/> <!-- Should a franka_gripper be mounted at the flange? (Currently does not work without it) -->
+  <xacro:arg name="special_connection" default=""/> <!-- Connection between the arm and the end-effector -->
   <xacro:property name="arm_id" value="$(arg arm_id)"/>
   <xacro:include filename="$(find franka_moveit_config)/srdf/panda_arm.xacro"/>
-  <xacro:panda_arm arm_id="${arm_id}"/>
+  <xacro:panda_arm arm_id="${arm_id}" special_connection="$(arg special_connection)"/>
   <xacro:if value="$(arg hand)">
     <xacro:include filename="$(find franka_moveit_config)/srdf/hand.xacro"/>
     <xacro:hand arm_id="${arm_id}"/>
     <xacro:include filename="$(find franka_moveit_config)/srdf/panda_arm_hand.xacro"/>
-    <xacro:panda_arm_hand arm_id="${arm_id}"/>
+    <xacro:panda_arm_hand arm_id="${arm_id}" special_connection="$(arg special_connection)"/>
   </xacro:if>
 </robot>

File: franka_moveit_config/srdf/panda_arm.xacro (robot description, xacro)
@@ -1,5 +1,5 @@
 <?xml version="1.0" ?>
 <robot xmlns:xacro="http://www.ros.org/wiki/xacro" name="panda">
-  <xacro:macro name="panda_arm" params="arm_id:='panda' ">
+  <xacro:macro name="panda_arm" params="arm_id:='panda' special_connection:='' ">
     <xacro:include filename="$(find franka_moveit_config)/srdf/group_definition.xacro"/>
     <xacro:group_definition arm_id="${arm_id}" group_name="${arm_id}_manipulator" tip_link="${arm_id}_hand_tcp"/>
@@ -28,4 +28,12 @@
     <disable_collisions link1="${arm_id}_link6" link2="${arm_id}_link8" reason="Default"/>
     <disable_collisions link1="${arm_id}_link7" link2="${arm_id}_link8" reason="Adjacent"/>
+    <xacro:unless value="${special_connection == ''}">
+      <disable_collisions link1="${arm_id}_link3" link2="${special_connection}" reason="Never"/>
+      <disable_collisions link1="${arm_id}_link4" link2="${special_connection}" reason="Never"/>
+      <disable_collisions link1="${arm_id}_link5" link2="${special_connection}" reason="Never"/>
+      <disable_collisions link1="${arm_id}_link6" link2="${special_connection}" reason="Never"/>
+      <disable_collisions link1="${arm_id}_link7" link2="${special_connection}" reason="Adjacent"/>
+      <disable_collisions link1="${arm_id}_link8" link2="${special_connection}" reason="Adjacent"/>
+    </xacro:unless>
   </xacro:macro>
 </robot>

File: franka_moveit_config/srdf/panda_arm_hand.xacro (robot description, xacro)
@@ -1,5 +1,5 @@
 <?xml version='1.0' encoding='utf-8'?>
 <robot xmlns:xacro="http://www.ros.org/wiki/xacro" name="panda">
-  <xacro:macro name="panda_arm_hand" params="arm_id:='panda' ">
+  <xacro:macro name="panda_arm_hand" params="arm_id:='panda' special_connection:='' ">
     <group_state name="open" group="hand">
       <joint name="${arm_id}_finger_joint1" value="0.035"/>
@@ -27,4 +27,9 @@
     <disable_collisions link1="${arm_id}_link7" link2="${arm_id}_rightfinger" reason="Never"/>
     <disable_collisions link1="${arm_id}_link8" link2="${arm_id}_rightfinger" reason="Never"/>
+    <xacro:unless value="${special_connection == ''}">
+      <disable_collisions link1="${arm_id}_hand" link2="${special_connection}" reason="Adjacent"/>
+      <disable_collisions link1="${arm_id}_leftfinger" link2="${special_connection}" reason="Never"/>
+      <disable_collisions link1="${arm_id}_rightfinger" link2="${special_connection}" reason="Never"/>
+    </xacro:unless>
   </xacro:macro>
 </robot>
