Commit message: implement collision behavior

File: franka_description/robots/panda_arm.ros2_control.xacro (robot description, xacro)
@@ -1,5 +1,5 @@
 <?xml version="1.0"?>
 <robot xmlns:xacro="http://www.ros.org/wiki/xacro">
-  <xacro:macro name="panda_arm_ros2_control" params="ns robot_ip use_fake_hardware:=^|false fake_sensor_commands:=^|false">
+  <xacro:macro name="panda_arm_ros2_control" params="ns robot_ip collision_behavior:='' use_fake_hardware:=^|false fake_sensor_commands:=^|false">
     <ros2_control name="FrankaHardwareInterface" type="system">
       <hardware>
@@ -12,4 +12,11 @@
           <plugin>franka_hardware/FrankaHardwareInterface</plugin>
           <param name="robot_ip">${robot_ip}</param>
+          <xacro:if value="${collision_behavior != ''}">
+            <xacro:property name="collision_thresholds" value="${xacro.load_yaml(collision_behavior)['collision_behavior']}"/>
+            <param name="lower_torque_thresholds">${' '.join(str(v) for v in collision_thresholds['lower_torque_thresholds'])}</param>
+            <param name="upper_torque_thresholds">${' '.join(str(v) for v in collision_thresholds['upper_torque_thresholds'])}</param>
+            <param name="lower_force_thresholds">${' '.join(str(v) for v in collision_thresholds['lower_force_thresholds'])}</param>
+            <param name="upper_force_thresholds">${' '.join(str(v) for v in collision_thresholds['upper_force_thresholds'])}</param>
+          </xacro:if>
         </xacro:unless>
       </hardware>

File: franka_description/robots/panda_arm.urdf.xacro (robot description, xacro)
@@ -3,4 +3,5 @@
   <xacro:arg name="arm_id" default="panda"/> <!-- Name of this panda -->
   <xacro:arg name="hand" default="false"/> <!-- Should a franka_gripper be mounted at the flange?" -->
+  <xacro:arg name="collision_behavior" default=""/>
   <xacro:arg name="robot_ip" default=""/> <!-- IP address or hostname of the robot" -->
   <xacro:arg name="use_fake_hardware" default="false"/>
@@ -49,4 +50,4 @@
   </xacro:if>
   <xacro:include filename="$(find franka_description)/robots/panda_arm.ros2_control.xacro"/>
-  <xacro:panda_arm_ros2_control ns="$(arg arm_id)" robot_ip="$(arg robot_ip)" use_fake_hardware="$(arg use_fake_hardware)" fake_sensor_commands="$(arg fake_sensor_commands)"/>
+  <xacro:panda_arm_ros2_control collision_behavior="$(arg collision_behavior)" ns="$(arg arm_id)" robot_ip="$(arg robot_ip)" use_fake_hardware="$(arg use_fake_hardware)" fake_sensor_commands="$(arg fake_sensor_commands)"/>
 </robot>

Commit message: implement cartesian impedance controller

File: franka_description/robots/panda_arm.ros2_control.xacro (robot description, xacro)
@@ -37,4 +37,15 @@
       <xacro:configure_joint joint_name="${ns}_joint6" initial_position="${pi/2}"/>
       <xacro:configure_joint joint_name="${ns}_joint7" initial_position="${pi/4}"/>
+      <xacro:macro name="configure_cartesian_velocity" params="axis">
+        <gpio name="${axis}">
+          <command_interface name="cartesian_velocity"/>
+        </gpio>
+      </xacro:macro>
+      <xacro:configure_cartesian_velocity axis="vx"/>
+      <xacro:configure_cartesian_velocity axis="vy"/>
+      <xacro:configure_cartesian_velocity axis="vz"/>
+      <xacro:configure_cartesian_velocity axis="wx"/>
+      <xacro:configure_cartesian_velocity axis="wy"/>
+      <xacro:configure_cartesian_velocity axis="wz"/>
     </ros2_control>
   </xacro:macro>
